Commit message: irc_table.stlの更新、tof_shapes.launch.pyで初期X位置を-0.25に変更、tof_robot.urdfでシリンダーの半径とジョイントの位置を調整

File: src/tof_sim/urdf/tof_robot.urdf (robot description, URDF)
Before this commit: robot tof_robot, 3 links, 2 joints
Links:
- link base_link: geometry collision cylinder length=0.12 radius=0.09; visual cylinder length=0.12 radius=0.09
Joints:
- joint tof_sensor_joint: origin xyz=0.17 0 0.14 rpy=0 0.261799 0 -> xyz=0.085 0 0.14 rpy=0 0.261799 0
